Commit message: update

File: src/husky_description/urdf/husky.urdf.xacro (robot description, xacro)
@@ -1,24 +1,3 @@
 <?xml version="1.0"?>
-<!--
-Software License Agreement (BSD)
-\file      husky.urdf.xacro
-\authors   Paul Bovbel <pbovbel@clearpathrobotics.com>, Devon Ash <dash@clearpathrobotics.com>
-\copyright Copyright (c) 2015, Clearpath Robotics, Inc., All rights reserved.
-Redistribution and use in source and binary forms, with or without modification, are permitted provided that
-the following conditions are met:
- * Redistributions of source code must retain the above copyright notice, this list of conditions and the
-   following disclaimer.
- * Redistributions in binary form must reproduce the above copyright notice, this list of conditions and the
-   following disclaimer in the documentation and/or other materials provided with the distribution.
- * Neither the name of Clearpath Robotics nor the names of its contributors may be used to endorse or promote
-   products derived from this software without specific prior written permission.
-THIS SOFTWARE IS PROVIDED BY THE COPYRIGHT HOLDERS AND CONTRIBUTORS "AS IS" AND ANY EXPRESS OR IMPLIED WAR-
-RANTIES, INCLUDING, BUT NOT LIMITED TO, THE IMPLIED WARRANTIES OF MERCHANTABILITY AND FITNESS FOR A PARTICULAR
-PURPOSE ARE DISCLAIMED. IN NO EVENT SHALL THE COPYRIGHT HOLDER OR CONTRIBUTORS BE LIABLE FOR ANY DIRECT, IN-
-DIRECT, INCIDENTAL, SPECIAL, EXEMPLARY, OR CONSEQUENTIAL DAMAGES (INCLUDING, BUT NOT LIMITED TO, PROCUREMENT
-OF SUBSTITUTE GOODS OR SERVICES; LOSS OF USE, DATA, OR PROFITS; OR BUSINESS INTERRUPTION) HOWEVER CAUSED AND
-ON ANY THEORY OF LIABILITY, WHETHER IN CONTRACT, STRICT LIABILITY, OR TORT (INCLUDING NEGLIGENCE OR OTHERWISE)
-ARISING IN ANY WAY OUT OF THE USE OF THIS SOFTWARE, EVEN IF ADVISED OF THE POSSIBILITY OF SUCH DAMAGE.
--->
 <robot name="husky" xmlns:xacro="http://ros.org/wiki/xacro">
   <xacro:arg name="laser_enabled" default="false" />
@@ -39,4 +18,6 @@
   <xacro:include filename="$(find husky_description)/urdf/accessories/sick_lms1xx_mount.urdf.xacro"/>
   <xacro:include filename="$(find husky_description)/urdf/accessories/sensor_arch.urdf.xacro"/>
+  <xacro:include filename="$(find ur_description)/urdf/ur5.urdf.xacro" />
+  <!-- <xacro:include filename="$(find husky_ur_description)/urdf/husky_ur5_description.urdf.xacro" /> -->
   <xacro:property name="M_PI" value="3.14159"/>
   <!-- Base Size -->
@@ -116,4 +97,15 @@
   </xacro:husky_wheel>
   <xacro:husky_decorate />
+  <xacro:if value="$(arg ur5_enabled)">
+    <xacro:property name="reflect" value="-1" />
+    <!-- Spawn arm -->
+    <xacro:ur5_robot prefix="ur5_arm_" joint_limited="true"/>
+    <!-- Join arm -->
+    <joint name="ur5_arm_base" type="fixed">
+      <parent link="top_plate_link" />
+      <child link="ur5_arm_base_link" />
+      <origin xyz="0.2 0 0.0065" rpy="0.0 0.0 -1.57" />
+    </joint>
+  </xacro:if>
   <xacro:if value="$(arg laser_enabled)">
     <xacro:sick_lms1xx_mount prefix="base"/>
